File: LaunchPad/4x4pad.brd (EAGLE design)
At the start: 127 x 101.6 mm, 33 parts

Commit message: Added double sided board
Routing:
- net GND: track 56.7 -> 0.00 mm
- net N$149: track 0.00 -> 11.5 mm
- net N$37: track 0.00 -> 5.56 mm
- removed copper zone on layer 1, net GND
Changed lines of the file:
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@@
 </class>
 </classes>
-<designrules name="default">
-<description language="de">&lt;b&gt;EAGLE Design Rules&lt;/b&gt;
-&lt;p&gt;
-Die Standard-Design-Rules sind so gewählt, dass sie für
-die meisten Anwendungen passen. Sollte ihre Platine
-besondere Anforderungen haben, treffen Sie die erforderlichen
-Einstellungen hier und speichern die Design Rules unter
-einem neuen Namen ab.</description>
-<description language="en">&lt;b&gt;EAGLE Design Rules&lt;/b&gt;
-&lt;p&gt;
-The default Design Rules have been set to cover
-a wide range of applications. Your particular design
-may have different requirements, so please make the
-necessary adjustments and save your customized
-design rules under a new name.</description>
+<designrules name="OthermillDRC_1_64_v2">
+<description language="en">&lt;b&gt;Othermill EAGLE Design Rules v2&lt;/b&gt;&lt;p&gt;DRC for Othermill, 1/64&quot; tool&lt;/p&gt;&lt;b&gt;-- Rules --&lt;/b&gt;&lt;li&gt;8 mil traces&lt;/li&gt;&lt;li&gt;15.7mil clearance&lt;/li&gt;</description>
 <param name="layerSetup" value="(1*16)"/>
 <param name="mtCopper" value="0.035mm 0.035mm 0.035mm 0.035mm 0.035mm 0.035mm 0.035mm 0.035mm 0.035mm 0.035mm 0.035mm 0.035mm 0.035mm 0.035mm 0.035mm 0.035mm"/>
 <param name="mtIsolate" value="1.5mm 0.15mm 0.2mm 0.15mm 0.2mm 0.15mm 0.2mm 0.15mm 0.2mm 0.15mm 0.2mm 0.15mm 0.2mm 0.15mm 0.2mm"/>
-<param name="mdWireWire" value="6mil"/>
-<param name="mdWirePad" value="6mil"/>
-<param name="mdWireVia" value="6mil"/>
-<param name="mdPadPad" value="6mil"/>
-<param name="mdPadVia" value="6mil"/>
-<param name="mdViaVia" value="6mil"/>
-<param name="mdSmdPad" value="6mil"/>
-<param name="mdSmdVia" value="6mil"/>
-<param name="mdSmdSmd" value="6mil"/>
-<param name="mdViaViaSameLayer" value="6mil"/>
+<param name="mdWireWire" value="0.39878125mm"/>
+<param name="mdWirePad" value="0.39878125mm"/>
+<param name="mdWireVia" value="0.39878125mm"/>
+<param name="mdPadPad" value="0.39878125mm"/>
+<param name="mdPadVia" value="0.39878125mm"/>
+<param name="mdViaVia" value="0.39878125mm"/>
+<param name="mdSmdPad" value="0mil"/>
+<param name="mdSmdVia" value="0mil"/>
+<param name="mdSmdSmd" value="0mil"/>
+<param name="mdViaViaSameLayer" value="8mil"/>
 <param name="mnLayersViaInSmd" value="2"/>
-<param name="mdCopperDimension" value="40mil"/>
-<param name="mdDrill" value="6mil"/>
+<param name="mdCopperDimension" value="0mil"/>
+<param name="mdDrill" value="1mil"/>
 <param name="mdSmdStop" value="0mil"/>
-<param name="msWidth" value="6mil"/>
-<param name="msDrill" value="0.35mm"/>
+<param name="msWidth" value="16mil"/>
+<param name="msDrill" value="31mil"/>
 <param name="msMicroVia" value="9.99mm"/>
 <param name="msBlindViaRatio" value="0.5"/>
@@
 <param name="rvMicroViaOuter" value="0.25"/>
 <param name="rvMicroViaInner" value="0.25"/>
-<param name="rlMinPadTop" value="10mil"/>
-<param name="rlMaxPadTop" value="20mil"/>
-<param name="rlMinPadInner" value="10mil"/>
-<param name="rlMaxPadInner" value="20mil"/>
-<param name="rlMinPadBottom" value="10mil"/>
-<param name="rlMaxPadBottom" value="20mil"/>
-<param name="rlMinViaOuter" value="8mil"/>
-<param name="rlMaxViaOuter" value="20mil"/>
+<param name="rlMinPadTop" value="0mil"/>
+<param name="rlMaxPadTop" value="9999mil"/>
+<param name="rlMinPadInner" value="0mil"/>
+<param name="rlMaxPadInner" value="9999mil"/>
+<param name="rlMinPadBottom" value="0mil"/>
+<param name="rlMaxPadBottom" value="9999mil"/>
+<param name="rlMinViaOuter" value="15mil"/>
+<param name="rlMaxViaOuter" value="25mil"/>
 <param name="rlMinViaInner" value="8mil"/>
-<param name="rlMaxViaInner" value="20mil"/>
+<param name="rlMaxViaInner" value="25mil"/>
 <param name="rlMinMicroViaOuter" value="4mil"/>
 <param name="rlMaxMicroViaOuter" value="20mil"/>
@@
 <param name="psBottom" value="-1"/>
 <param name="psFirst" value="-1"/>
-<param name="psElongationLong" value="100"/>
+<param name="psElongationLong" value="50"/>
 <param name="psElongationOffset" value="100"/>
-<param name="mvStopFrame" value="1"/>
-<param name="mvCreamFrame" value="0"/>
-<param name="mlMinStopFrame" value="4mil"/>
-<param name="mlMaxStopFrame" value="4mil"/>
-<param name="mlMinCreamFrame" value="0mil"/>
-<param name="mlMaxCreamFrame" value="0mil"/>
-<param name="mlViaStopLimit" value="0mil"/>
-<param name="srRoundness" value="0"/>
-<param name="srMinRoundness" value="0mil"/>
-<param name="srMaxRoundness" value="0mil"/>
+<param name="mvStopFrame" value="0.05"/>
+<param name="mvCreamFrame" value="0.05"/>
+<param name="mlMinStopFrame" value="1mil"/>
+<param name="mlMaxStopFrame" value="2mil"/>
+<param name="mlMinCreamFrame" value="2mil"/>
+<param name="mlMaxCreamFrame" value="10mil"/>
+<param name="mlViaStopLimit" value="30mil"/>
+<param name="srRoundness" value="0.1"/>
+<param name="srMinRoundness" value="2mil"/>
+<param name="srMaxRoundness" value="10mil"/>
 <param name="slThermalIsolate" value="10mil"/>
 <param name="slThermalsForVias" value="0"/>
@@
 <vertex x="127" y="104.14"/>
 </polygon>
-</signal>
-<signal name="GND">
 <polygon width="0.1524" layer="1">
 <vertex x="24" y="98"/>
@@
 </polygon>
 <wire x1="25.4" y1="99" x2="25.4" y2="95" width="1" layer="1"/>
-<wire x1="6.3" y1="45.6" x2="11.2" y2="45.6" width="0.125" layer="1"/>
-<wire x1="11.2" y1="45.6" x2="12.6" y2="47" width="0.125" layer="1"/>
-<wire x1="12.6" y1="47" x2="12.6" y2="81.1" width="0.125" layer="1"/>
-<wire x1="12.7" y1="94" x2="15.9" y2="94" width="0.1524" layer="1"/>
-<wire x1="15.9" y1="94" x2="21.9" y2="88" width="0.1524" layer="1"/>
-<wire x1="21.9" y1="88" x2="25.4" y2="95" width="0" layer="19" extent="1-1"/>
-<wire x1="12.6" y1="81.1" x2="21.9" y2="88" width="0" layer="19" extent="1-1"/>
+<wire x1="6.9" y1="45.1" x2="8" y2="44" width="0.1524" layer="1"/>
+<wire x1="35.35" y1="89.7162" x2="25.4" y2="95" width="0" layer="19" extent="1-1"/>
+<wire x1="12.7" y1="96.52" x2="25.4" y2="95" width="0" layer="19" extent="1-1"/>
+<wire x1="111.55" y1="64.3162" x2="111.55" y2="89.7162" width="0" layer="19" extent="1-1"/>
+<wire x1="111.55" y1="38.9162" x2="111.55" y2="13.5162" width="0" layer="19" extent="1-1"/>
+<wire x1="86.15" y1="38.9162" x2="111.55" y2="38.9162" width="0" layer="19" extent="1-1"/>
+<wire x1="60.75" y1="38.9162" x2="86.15" y2="38.9162" width="0" layer="19" extent="1-1"/>
+<wire x1="86.15" y1="64.3162" x2="86.15" y2="89.7162" width="0" layer="19" extent="1-1"/>
+<wire x1="60.75" y1="64.3162" x2="60.75" y2="89.7162" width="0" layer="19" extent="1-1"/>
+<wire x1="35.35" y1="64.3162" x2="35.35" y2="89.7162" width="0" layer="19" extent="1-1"/>
+<wire x1="60.75" y1="13.5162" x2="35.35" y2="13.5162" width="0" layer="19" extent="1-1"/>
+<wire x1="86.15" y1="13.5162" x2="111.55" y2="13.5162" width="0" layer="19" extent="1-1"/>
+<wire x1="35.35" y1="38.9162" x2="35.35" y2="13.5162" width="0" layer="19" extent="1-1"/>
 </signal>
 <signal name="N$41">
@@
 <wire x1="20.9" y1="86.4" x2="21.7" y2="85.6" width="0.1524" layer="1"/>
 </signal>
+<signal name="N$149">
+<wire x1="12.7" y1="93.9" x2="15.9" y2="93.9" width="0.1524" layer="1"/>
+<wire x1="15.9" y1="93.9" x2="21.8" y2="88" width="0.1524" layer="1"/>
+</signal>
 </signals>
